File: PCB_Design/TransmitterSide/TransmitterPCB/TransmitterPCB.kicad_pcb (KiCad board)
At the start: 2 copper layers, 8 parts, among them J1 Conn_01x02_Pin, U1 PAM8302AAY

Commit message: Transmitter PCB finished... maybe
Parts:
- added H1: MountingHole, MountingHole:MountingHole_3.2mm_M3, F.Cu at (109.5, 51.5)
- added H2: MountingHole, MountingHole:MountingHole_3.2mm_M3, F.Cu at (156.0, 51.5)
- added H3: MountingHole, MountingHole:MountingHole_3.2mm_M3, F.Cu at (156.0, 110.5)
- added H4: MountingHole, MountingHole:MountingHole_3.2mm_M3, F.Cu at (109.5, 110.5)
Routing:
- added copper zone on B.Cu, net GND
Other:
- board outline added: 63 x 72.5 mm
