File: PCB_Design/TransmitterSide/TransmitterPCB/TransmitterPCB.kicad_sch (KiCad schematic)
At the start: 8 parts, among them J1 Conn_01x02_Pin, U1 PAM8302AAY

Commit message: Transmitter PCB finished... maybe
Parts:
- added H1, H2, H3, H4: MountingHole, MountingHole:MountingHole_3.2mm_M3, symbol Mechanical:MountingHole
