File: PCB_Design/ReceiverSide/ReceiverSide.kicad_sch (KiCad schematic)
At the start: 15 parts, among them J1 Conn_01x02_Pin, U1 DRV5053CAQLPGM

Commit message: some edits on receiver side
Parts:
- removed R6: R, Resistor_THT:R_Axial_DIN0204_L3.6mm_D1.6mm_P1.90mm_Vertical, symbol Device:R
- renumbered D4 to D1, D3 to D2, D2 to D3, D1 to D4
Connections:
- net Speaker is gone; now on net D6: LS1.1
- net GND: now also D1.1 (K), D2.1 (K), D3.1 (K), D4.1 (K); no longer D1.2 (A), D2.2 (A), D3.2 (A), D4.2 (A)
- net LEDa: now also D1.2 (A); no longer D4.1 (K)
- net LEDb: now also D2.2 (A); no longer D3.1 (K)
- net LEDc: now also D3.2 (A); no longer D2.1 (K)
- net LEDd: now also D4.2 (A); no longer D1.1 (K)
Other:
- moved on the sheet: D1, D2, D3, D4
Changed lines of the file:
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@@
-		)
-	)
-	(label "Speaker"
-		(at 54.61 138.43 180)
-		(effects
-			(font
-				(size 1.27 1.27)
-			)
-			(justify right bottom)
-		)
-	)
-	(label "Speaker"
-		(at 69.85 139.7 180)
-		(effects
-			(font
-				(size 1.27 1.27)
-			)
-			(justify right bottom)
 		)
 	)
@@
 		)
 	)
-	(label "D6"
-		(at 54.61 146.05 270)
-		(effects
-			(font
-				(size 1.27 1.27)
-			)
-			(justify right bottom)
-		)
-	)
 	(label "LED1"
 		(at 113.03 92.71 180)
@@
 		)
 	)
+	(label "D6"
+		(at 69.85 139.7 180)
+		(effects
+			(font
+				(size 1.27 1.27)
+			)
+			(justify right bottom)
+		)
+	)
 	(label "LEDc"
 		(at 86.36 128.27 270)
@@
 	(symbol
 		(lib_id "Device:LED")
-		(at 97.79 105.41 0)
-		(unit 1)
-		(exclude_from_sim no)
-		(in_bom yes)
-		(on_board yes)
-		(dnp no)
-		(fields_autoplaced yes)
-		(property "Reference" "D3"
-			(at 96.2025 99.06 0)
+		(at 80.01 91.44 180)
+		(unit 1)
+		(exclude_from_sim no)
+		(in_bom yes)
+		(on_board yes)
+		(dnp no)
+		(property "Reference" "D2"
+			(at 80.518 94.742 0)
 			(effects
 				(font
@@
 		)
 		(property "Value" "LED"
-			(at 96.2025 101.6 0)
+			(at 80.772 87.63 0)
 			(effects
 				(font
@@
 		)
 		(property "Footprint" "LED_THT:LED_D3.0mm"
-			(at 97.79 105.41 0)
+			(at 80.01 91.44 0)
 			(effects
 				(font
@@
 		)
 		(property "Datasheet" "~"
-			(at 97.79 105.41 0)
+			(at 80.01 91.44 0)
 			(effects
 				(font
@@
 		)
 		(property "Description" "Light emitting diode"
-			(at 97.79 105.41 0)
+			(at 80.01 91.44 0)
 			(effects
 				(font
@@
 		)
 		(property "Sim.Pins" "1=K 2=A"
-			(at 97.79 105.41 0)
+			(at 80.01 91.44 0)
 			(effects
 				(font
@@
 			(project "ReceiverSide"
 				(path "/36cd22f2-71f9-449d-86c3-0d6a26eca8a0"
-					(reference "D3")
+					(reference "D2")
 					(unit 1)
 				)
@@
 	(symbol
 		(lib_id "Device:LED")
-		(at 80.01 105.41 0)
-		(unit 1)
-		(exclude_from_sim no)
-		(in_bom yes)
-		(on_board yes)
-		(dnp no)
-		(fields_autoplaced yes)
+		(at 97.79 91.44 180)
+		(unit 1)
+		(exclude_from_sim no)
+		(in_bom yes)
+		(on_board yes)
+		(dnp no)
+		(property "Reference" "D1"
+			(at 97.536 93.726 0)
+			(effects
+				(font
+					(size 1.27 1.27)
+				)
+			)
+		)
+		(property "Value" "LED"
+			(at 98.552 87.63 0)
+			(effects
+				(font
+					(size 1.27 1.27)
+				)
+			)
+		)
+		(property "Footprint" "LED_THT:LED_D3.0mm"
+			(at 97.79 91.44 0)
+			(effects
+				(font
+					(size 1.27 1.27)
+				)
+				(hide yes)
+			)
+		)
+		(property "Datasheet" "~"
+			(at 97.79 91.44 0)
+			(effects
+				(font
+					(size 1.27 1.27)
+				)
+				(hide yes)
+			)
+		)
+		(property "Description" "Light emitting diode"
+			(at 97.79 91.44 0)
+			(effects
+				(font
+					(size 1.27 1.27)
+				)
+				(hide yes)
+			)
+		)
+		(property "Sim.Pins" "1=K 2=A"
+			(at 97.79 91.44 0)
+			(effects
+				(font
+					(size 1.27 1.27)
+				)
+				(hide yes)
+			)
+		)
+		(pin "1"
+		)
+		(pin "2"
+		)
+		(instances
+			(project "ReceiverSide"
+				(path "/36cd22f2-71f9-449d-86c3-0d6a26eca8a0"
+					(reference "D1")
+					(unit 1)
+				)
+			)
+		)
+	)
+	(symbol
+		(lib_id "Device:LED")
+		(at 80.01 105.41 180)
+		(unit 1)
+		(exclude_from_sim no)
+		(in_bom yes)
+		(on_board yes)
+		(dnp no)
 		(property "Reference" "D4"
-			(at 78.4225 99.06 0)
+			(at 80.264 108.712 0)
 			(effects
 				(font
@@
 		)
 		(property "Value" "LED"
-			(at 78.4225 101.6 0)
+			(at 80.518 101.854 0)
 			(effects
 				(font
@@
 		)
 		(instances
-			(project "ReceiverSide"
+			(project ""
 				(path "/36cd22f2-71f9-449d-86c3-0d6a26eca8a0"
 					(reference "D4")
-					(unit 1)
-				)
-			)
-		)
-	)
-	(symbol
-		(lib_id "Device:LED")
-		(at 97.79 91.44 0)
-		(unit 1)
-		(exclude_from_sim no)
-		(in_bom yes)
-		(on_board yes)
-		(dnp no)
-		(fields_autoplaced yes)
-		(property "Reference" "D1"
-			(at 96.2025 85.09 0)
-			(effects
-				(font
-					(size 1.27 1.27)
-				)
-			)
-		)
-		(property "Value" "LED"
-			(at 96.2025 87.63 0)
-			(effects
-				(font
-					(size 1.27 1.27)
-				)
-			)
-		)
-		(property "Footprint" "LED_THT:LED_D3.0mm"
-			(at 97.79 91.44 0)
-			(effects
-				(font
-					(size 1.27 1.27)
-				)
-				(hide yes)
-			)
-		)
-		(property "Datasheet" "~"
-			(at 97.79 91.44 0)
-			(effects
-				(font
-					(size 1.27 1.27)
-				)
-				(hide yes)
-			)
-		)
-		(property "Description" "Light emitting diode"
-			(at 97.79 91.44 0)
-			(effects
-				(font
-					(size 1.27 1.27)
-				)
-				(hide yes)
-			)
-		)
-		(property "Sim.Pins" "1=K 2=A"
-			(at 97.79 91.44 0)
-			(effects
-				(font
-					(size 1.27 1.27)
-				)
-				(hide yes)
-			)
-		)
-		(pin "1"
-		)
-		(pin "2"
-		)
-		(instances
-			(project ""
-				(path "/36cd22f2-71f9-449d-86c3-0d6a26eca8a0"
-					(reference "D1")
 					(unit 1)
 				)
@@
 	(symbol
 		(lib_id "Device:R")
-		(at 54.61 142.24 0)
-		(unit 1)
-		(exclude_from_sim no)
-		(in_bom yes)
-		(on_board yes)
-		(dnp no)
-		(fields_autoplaced yes)
-		(property "Reference" "R6"
-			(at 57.15 140.9699 0)
-			(effects
-				(font
-					(size 1.27 1.27)
-				)
-				(justify left)
-			)
-		)
-		(property "Value" "R"
-			(at 57.15 143.5099 0)
-			(effects
-				(font
-					(size 1.27 1.27)
-				)
-				(justify left)
-			)
-		)
-		(property "Footprint" "Resistor_THT:R_Axial_DIN0204_L3.6mm_D1.6mm_P1.90mm_Vertical"
-			(at 52.832 142.24 90)
-			(effects
-				(font
-					(size 1.27 1.27)
-				)
-				(hide yes)
-			)
-		)
-		(property "Datasheet" "~"
-			(at 54.61 142.24 0)
-			(effects
-				(font
-					(size 1.27 1.27)
-				)
-				(hide yes)
-			)
-		)
-		(property "Description" "Resistor"
-			(at 54.61 142.24 0)
-			(effects
-				(font
-					(size 1.27 1.27)
-				)
-				(hide yes)
-			)
-		)
-		(pin "2"
-		)
-		(pin "1"
-		)
-		(instances
-			(project "ReceiverSide"
-				(path "/36cd22f2-71f9-449d-86c3-0d6a26eca8a0"
-					(reference "R6")
-					(unit 1)
-				)
-			)
-		)
-	)
-	(symbol
-		(lib_id "Device:R")
 		(at 172.72 119.38 0)
 		(unit 1)
@@
 	(symbol
 		(lib_id "Device:LED")
-		(at 80.01 91.44 0)
-		(unit 1)
-		(exclude_from_sim no)
-		(in_bom yes)
-		(on_board yes)
-		(dnp no)
-		(fields_autoplaced yes)
-		(property "Reference" "D2"
-			(at 78.4225 85.09 0)
+		(at 97.79 105.41 180)
+		(unit 1)
+		(exclude_from_sim no)
+		(in_bom yes)
+		(on_board yes)
+		(dnp no)
+		(property "Reference" "D3"
+			(at 99.06 108.966 0)
 			(effects
 				(font
@@
 		)
 		(property "Value" "LED"
-			(at 78.4225 87.63 0)
+			(at 98.044 102.362 0)
 			(effects
 				(font
@@
 		)
 		(property "Footprint" "LED_THT:LED_D3.0mm"
-			(at 80.01 91.44 0)
+			(at 97.79 105.41 0)
 			(effects
 				(font
@@
 		)
 		(property "Datasheet" "~"
-			(at 80.01 91.44 0)
+			(at 97.79 105.41 0)
 			(effects
 				(font
@@
 		)
 		(property "Description" "Light emitting diode"
-			(at 80.01 91.44 0)
+			(at 97.79 105.41 0)
 			(effects
 				(font
@@
 		)
 		(property "Sim.Pins" "1=K 2=A"
-			(at 80.01 91.44 0)
+			(at 97.79 105.41 0)
 			(effects
 				(font
@@
 			(project "ReceiverSide"
 				(path "/36cd22f2-71f9-449d-86c3-0d6a26eca8a0"
-					(reference "D2")
-					(unit 1)
-				)
+					(reference "D3")
+					(unit 1)
+				)

Commit message: COMPLETED RECIVER PCB
Parts:
- removed J1: Conn_01x02_Pin, Connector_PinHeader_1.27mm:PinHeader_1x02_P1.27mm_Vertical, symbol Connector:Conn_01x02_Pin
- removed LS1: Speaker, Resistor_THT:R_Axial_DIN0204_L3.6mm_D1.6mm_P1.90mm_Vertical, symbol Device:Speaker
- removed U1: DRV5053CAQLPGM, Halleffect:LPG3_TEX, symbol HallEffect:DRV5053CAQLPGM
- added ACC1, ACC2, ACC3, ACC4, ACC5: R, Resistor_THT:R_Axial_DIN0204_L3.6mm_D1.6mm_P5.08mm_Horizontal, symbol Device:R
- added AUX-PWR1, Hall1, OP-IN1, OP-PWR1, Speaker1: Conn_01x02_Socket, Connector_PinSocket_2.54mm:PinSocket_1x02_P2.54mm_Vertical, symbol Connector:Conn_01x02_Socket
- added H1, H2, H3, H4: MountingHole, MountingHole:MountingHole_2.7mm, symbol Mechanical:MountingHole
- added HALL-IN1, OP-OUT1: Conn_01x01_Socket, Connector_PinSocket_2.54mm:PinSocket_1x01_P2.54mm_Vertical, symbol Connector:Conn_01x01_Socket
- added Op-Amp1: MCP6281-E_P, MCP6281_E_P:DIP787W46P254L927H533Q8, symbol MCP6281-E_P:MCP6281-E_P
- PR1: renamed from R9; footprint Resistor_THT:R_Axial_DIN0204_L3.6mm_D1.6mm_P1.90mm_Vertical -> Resistor_THT:R_Axial_DIN0204_L3.6mm_D1.6mm_P5.08mm_Horizontal
- R1, R2, R3, R4, R5: footprint Resistor_THT:R_Axial_DIN0204_L3.6mm_D1.6mm_P1.90mm_Vertical -> Resistor_THT:R_Axial_DIN0204_L3.6mm_D1.6mm_P5.08mm_Horizontal
- renumbered D4 to D1, D3 to D2, D2 to D3, D1 to D4
Connections:
- net +5V: now also Hall1.1 (Pin_1)
- net GND: now also AUX-PWR1.1 (Pin_1), Hall1.2 (Pin_2), Speaker1.2 (Pin_2)
- net Halleffect: now also HALL-IN1.1 (Pin_1)
- net at A1.30 (VIN): now also AUX-PWR1.2 (Pin_2)
- net D6 renamed Speaker
- net Speaker: now also Speaker1.1 (Pin_1)
- net LEDa: no longer names the net of R1.2
- net LEDa: now also D1.2 (A); no longer D4.2 (A)
- net LEDb: no longer names the net of D3.2 (A)
- net LEDb: now also R3.2; no longer R2.2
- net LEDc: no longer names the net of D2.2 (A)
- net LEDc: now also R2.2; no longer R3.2
- net LEDd: no longer names the net of R4.2
- net LEDd: now also D4.2 (A); no longer D1.2 (A)
- new net: ACC4.1, OP-IN1.1 (Pin_1)
- new net: ACC3.2, OP-IN1.2 (Pin_2)
- new net: ACC1.2, ACC2.2
- new net: ACC4.2, ACC5.2, Op-Amp1.2 (VIN-)
- new net: ACC3.1, Op-Amp1.3 (VIN+)
- new net VDD+: OP-PWR1.2 (Pin_2), Op-Amp1.7 (VDD)
- new net VOUT: ACC5.1, OP-OUT1.1 (Pin_1), Op-Amp1.6 (VOUT)
- new net VSS-: OP-PWR1.1 (Pin_1), Op-Amp1.4 (VSS)
- no-connect marks 19 -> 22
Other:
- moved on the sheet: A1, D1, D2, D3, D4, PR1, R5

Commit message: PCB DONE
Parts:
- added GND1, GND2: Conn_01x01_Socket, Connector_PinSocket_2.54mm:PinSocket_1x01_P2.54mm_Vertical, symbol Connector:Conn_01x01_Socket
- added OP-PWR-IN1: Conn_01x02_Socket, Connector_PinSocket_2.54mm:PinSocket_1x02_P2.54mm_Vertical, symbol Connector:Conn_01x02_Socket
Connections:
- net +5V: now also OP-PWR-IN1.1 (Pin_1)
- net GND: now also GND1.1 (Pin_1), GND2.1 (Pin_1)
- net +3.3V: now reaches A1.17 (3V3)
- net +3.3V: now also OP-PWR-IN1.2 (Pin_2)
- no-connect marks 22 -> 21
Other:
- moved on the sheet: Hall1, PR1, R5
